File: Nailem-Main-PCB/Nailem.kicad_pcb (KiCad board)
At the start: 2 copper layers, 95 x 95 mm, 118 parts, among them J1 USB_OTG, J10 LED_CH4, J11 12VIN, J12 J_SR04, J13 J_DS18B20_1, J14 J_DS18B20_2, J15 J_DS18B20_3, J16 J_DS18B20_4, J17 J_STATUS, J18 J_SERVO, J19 J_TURBIDITY, J2 J_UART, J20 5VIN, J21 J_TDS, J22 J_PH, J23 J_STEPPER, J24 J_5V_LCD, J25 J_5V_NEXTION, J26 J_3V3_LUX, J27 J_SERVO2, J28 J_ENDS, J29 5VPI, J3 OUT_CH1, J4 OUT_CH2, J5 OUT_CH3, J6 OUT_CH4, J7 LED_CH1, J8 LED_CH2, J9 LED_CH3, K1 SANYOU_SRD_Form_C, K2 SANYOU_SRD_Form_C, K3 SANYOU_SRD_Form_C, K4 SANYOU_SRD_Form_C, Q1 MMBT2222A, Q2 MMBT2222A, Q3 MMBT2222A, Q4 MMBT2222A, Q5 AON6980, Q6 AON6980, Q7 AON6980, Q8 AON6980, SW1 SW_SPST, SW2 SW_SPST, SW3 SW_DIP_x03, U1 ESP32-S3-WROOM-1, U2 AMS1117-3.3, U3 INA3221_Module

Commit message: Finalize PCB
PCB complete, and is currently being produced under JLCPCB with files in 'Production files for PCB'
Parts:
- added G***: LOGO, LOGO, F.Cu at (233.8, 91.5)
- added G***: LOGO, LOGO, F.Cu at (239.5, 140.7)
- added G***: LOGO, LOGO, F.Cu at (222.2, 119.0)
- added G***: LOGO, LOGO, F.Cu at (203.1, 128.5)
- added G***: LOGO, LOGO, F.Cu at (240.5, 91.8)
- added G***: LOGO, LOGO, F.Cu at (257.8, 135.5)
- added G***: LOGO, LOGO, F.Cu at (250.8, 58.5)
- added G***: LOGO, LOGO, F.Cu at (212.7, 65.2)
- added G***: LOGO, LOGO, F.Cu at (203.1, 94.5)
- added G***: LOGO, LOGO, F.Cu at (175.5, 84.2)
- added G***: LOGO, LOGO, F.Cu at (246.8, 106.0)
- added G***: LOGO, LOGO, F.Cu at (211.6, 137.0)
- added G***: LOGO, LOGO, F.Cu at (240.8, 106.5)
- added G***: LOGO, LOGO, F.Cu at (229.0, 138.4)
- added G***: LOGO, LOGO, F.Cu at (175.5, 117.8)
- added G***: LOGO, LOGO, F.Cu at (237.2, 68.0)
- added G***: LOGO, LOGO, F.Cu at (198.0, 67.2)
- added G***: LOGO, LOGO, F.Cu at (175.5, 134.8)
- added G***: LOGO, LOGO, F.Cu at (233.8, 119.0)
- added G***: LOGO, LOGO, F.Cu at (187.1, 143.1)
- added G***: LOGO, LOGO, F.Cu at (208.2, 78.5)
- added G***: LOGO, LOGO, F.Cu at (226.5, 65.2)
- added G***: LOGO, LOGO, F.Cu at (203.1, 78.0)
- added G***: LOGO, LOGO, F.Cu at (211.0, 119.0)
- added G***: LOGO, LOGO, B.Cu at (227.3, 120.0)
- added G***: LOGO, LOGO, B.Cu at (230.9, 70.9)
- added G***: LOGO, LOGO, B.Cu at (189.0, 57.2)
- added G***: LOGO, LOGO, F.Cu at (233.8, 99.0)
- added G***: LOGO, LOGO, F.Cu at (252.1, 124.8)
- added G***: LOGO, LOGO, F.Cu at (208.2, 71.5)
- added G***: LOGO, LOGO, F.Cu at (175.5, 100.8)
- added G***: LOGO, LOGO, F.Cu at (203.1, 111.5)
- added G***: LOGO, LOGO, F.Cu at (185.0, 67.2)
- C12, C7, R20, R21, R22, R23, R24, R25, R26, R27, R28, R29, R30, R4, R41, R42: moved to B.Cu
- D10, D3, D6, D8: footprint Diode_SMD:D_SMA-SMB_Universal_Handsoldering -> Custom_Footprints:D_SMA-SMB_Universal_Handsoldering_NoSilk
- J10, J7, J8, J9: footprint TerminalBlock:TerminalBlock_Xinya_XY308-2.54-2P_1x02_P2.54mm_Horizontal -> Custom_Footprints:TerminalBlock_Xinya_XY308-2.54-2P_1x02_P2.54mm_Horizontal_NoTriangle
- J11, J20, J3, J4, J5, J6: footprint Custom_Footprints:2EDGK_5.08_2P_M -> Custom_Footprints:2EDGK_5.08_2P_M_NEW
- K1, K2, K3, K4: footprint Relay_THT:Relay_SPDT_SANYOU_SRD_Series_Form_C -> Custom_Footprints:Relay_SPDT_SANYOU_SRD_Series_Form_C_NoInSilk
- Q5, Q6, Q7, Q8: footprint PCM_Package_SON_AKL:Infineon_PG-TISON-8-2 -> Custom_Footprints:SO-8FL_DFN5x6; moved to B.Cu
- SW1: value SW_SPST -> SW_RST; footprint Button_Switch_THT:SW_PUSH_6mm -> Button_Switch_SMD:SW_SPST_TS-1088-xR020
- SW2: value SW_SPST -> SW_BOOT; footprint Button_Switch_THT:SW_PUSH_6mm -> Button_Switch_SMD:SW_SPST_TS-1088-xR020
- moved Q8 77.6 mm to (203.4, 138.5), turned to 90 degrees
- moved R27 72.8 mm to (202.0, 133.0), turned to 90 degrees
- moved R26 68.5 mm to (205.0, 133.0), turned to -90 degrees
- moved Q7 68.0 mm to (210.3, 138.5), turned to 90 degrees
- moved R25 63.6 mm to (209.2, 133.0), turned to 90 degrees
- moved R42 61.1 mm to (246.5, 94.0), turned to 180 degrees
- moved R24 59.4 mm to (212.2, 133.0), turned to -90 degrees
- moved Q6 58.5 mm to (217.1, 138.5), turned to 90 degrees
- moved R41 55.7 mm to (246.5, 97.0), turned to 180 degrees
- moved R23 54.8 mm to (215.7, 133.0), turned to 90 degrees
- moved R22 50.6 mm to (218.7, 133.0), turned to -90 degrees
- moved Q5 49.0 mm to (224.0, 138.5), turned to 90 degrees
- moved C10 47.6 mm to (210.1, 125.5), turned to 0 degrees
- moved J23 47.3 mm to (250.3, 139.1), turned to 90 degrees
- moved R21 44.3 mm to (225.9, 133.0), turned to -90 degrees
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Connections:
- J28 pad 1: END_XPLUS -> END_XMIN
- J28 pad 2: END_XMIN -> END_XPLUS
- R28 pad 1: HCSR04_ECHO -> Net-(J12-Pin_4)
- R28 pad 2: Net-(J12-Pin_4) -> HCSR04_ECHO
- R41 pad 2: END_XMIN -> END_XPLUS
- R42 pad 2: END_XPLUS -> END_XMIN
Routing:
- net 3V3LOGIC: track 117.6 -> 222.4 mm, vias 2 -> 3
- net LED_DRV_CH4: track 28.1 -> 106.6 mm, vias 0 -> 5
- net IND_ARGB: track 5.61 -> 82.9 mm, vias 0 -> 3
- net LED_DRV_CH3: track 8.96 -> 74.9 mm, vias 1 -> 3
- net STEP_STP: track 4.14 -> 57.3 mm, vias 0 -> 4
- net Net-(SW1-B): track 29.1 -> 65.8 mm, vias 3 -> 5
- net Net-(SW2-B): track 4.66 -> 39.7 mm, vias 1 -> 2
- net STEP_EN: track 9.80 -> 42.4 mm, vias 0 -> 3
- net LED_DRV_CH2: track 37.6 -> 67.8 mm, vias 0 -> 3
- net STEP_DIR: track 27.6 -> 57.6 mm, vias 0 -> 1
- net LED_DRV_CH1: track 36.3 -> 64.4 mm, vias 0 -> 3
- net GND: track 217.3 -> 233.6 mm, vias 22 -> 548
- net RELAY_CH4: track 116.4 -> 103.2 mm
- net RELAY_CH3: track 100.3 -> 87.1 mm
- net Net-(A1-MS1): track 19.2 -> 7.61 mm
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- added copper zone on F.Cu, net 12V
- added copper zone on F.Cu, net GND
Other:
- outline, holes or cut-outs redrawn
