File: Nailem-Main-PCB/test.kicad_sch (KiCad schematic)
At the start: 26 parts, among them J1 USB_OTG, J2 J_UART, SW1 SW_SPST, SW2 SW_SPST, U1 ESP32-S3-WROOM-1, U2 AMS1117-3.3

Commit message: Finalize PCB
PCB complete, and is currently being produced under JLCPCB with files in 'Production files for PCB'
Parts:
- SW1: value SW_SPST -> SW_RST; footprint Button_Switch_THT:SW_PUSH_6mm -> Button_Switch_SMD:SW_SPST_TS-1088-xR020
- SW2: value SW_SPST -> SW_BOOT; footprint Button_Switch_THT:SW_PUSH_6mm -> Button_Switch_SMD:SW_SPST_TS-1088-xR020
Changed lines of the file:
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@@
 			)
 		)
-		(property "Value" "SW_SPST"
+		(property "Value" "SW_RST"
 			(at 87.63 120.65 0)
 			(show_name no)
@@
 			)
 		)
-		(property "Footprint" "Button_Switch_THT:SW_PUSH_6mm"
+		(property "Footprint" "Button_Switch_SMD:SW_SPST_TS-1088-xR020"
 			(at 87.63 124.46 0)
 			(hide yes)
@@
 			)
 		)
-		(property "Value" "SW_SPST"
+		(property "Value" "SW_BOOT"
 			(at 87.63 130.81 0)
 			(show_name no)
@@
 			)
 		)
-		(property "Footprint" "Button_Switch_THT:SW_PUSH_6mm"
+		(property "Footprint" "Button_Switch_SMD:SW_SPST_TS-1088-xR020"
 			(at 87.63 134.62 0)
 			(hide yes)
